File: TGS2600/TGS2600.kicad_sch (KiCad schematic)
At the start: 5 parts, among them J1 Conn_01x05_Pin

Commit message: Update for manufacturing
Parts:
- R1, R2: footprint fab:R_1206 -> Resistor_SMD:R_1206_3216Metric
Changed lines of the file:
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@@
 			)
 		)
-		(property "Footprint" "fab:R_1206"
+		(property "Footprint" "Resistor_SMD:R_1206_3216Metric"
 			(at 109.22 109.22 90)
 			(effects
@@
 			)
 		)
-		(property "Footprint" "fab:R_1206"
+		(property "Footprint" "Resistor_SMD:R_1206_3216Metric"
 			(at 109.22 88.9 90)
 			(effects
