File: TGS2600/TGS2600.kicad_pcb (KiCad board)
At the start: 2 copper layers, 28.8 x 40.6 mm, 5 parts, among them J1 Conn_01x05_Pin

Commit message: Update for manufacturing
Parts:
- added H1: MountingHole, MountingHole:MountingHole_3.2mm_M3_DIN965_Pad, F.Cu at (2102.1, 2115.1)
- added H2: MountingHole, MountingHole:MountingHole_3.2mm_M3_DIN965_Pad, F.Cu at (2102.1, 2113.5)
- added REF**: OSHW-Logo2_7.3x6mm_SilkScreen, Symbol:OSHW-Logo2_7.3x6mm_SilkScreen, F.Cu at (135.7, 85.1)
- R1, R2: footprint fab:R_1206 -> Resistor_SMD:R_1206_3216Metric
- moved R1 17.8 mm to (156.7, 89.9)
- moved R2 17.8 mm to (156.7, 107.6)
- moved U1 17.8 mm to (147.3, 86.9)
- moved U2 17.8 mm to (147.3, 104.7)
Routing:
- net Vout1: track 43.1 -> 29.6 mm, vias 1 -> 0
- net GND: track 81.9 -> 94.4 mm, vias 1 -> 0
- net Vin: track 47.6 -> 37.5 mm, vias 1 -> 0
- net Vout2: track 30.9 -> 35.4 mm, vias 1 -> 0
Other:
- board text added: "S1"
- board text added: "S2"
- board text added: "Smart Citizen Fab Lab Barcelona"
- board text added: "V+"
- board text added: "V-"
- board text added: "VOC Sensor Board V0.1"

Commit message: Fix mounting holes preventing manufacturing
Parts:
- removed H1, H2: MountingHole, MountingHole:MountingHole_3.2mm_M3_DIN965_Pad
- moved R1 10.8 mm to (150.1, 81.3)
- moved R2 10.8 mm to (150.1, 99.1)
- moved J1 10.8 mm to (130.5, 85.4)
- moved REF** 10.8 mm to (129.0, 76.6)
- moved U1 10.8 mm to (140.7, 78.4)
- moved U2 10.8 mm to (140.7, 96.2)
